File: card.brd (EAGLE design)
At the start: 160 x 100 mm, 33 parts, among them J1 5-PIN_2MM-V, J2 B2PS-VH(LF)(SN), U3 TLV70233DBVR, X1 MINI-USB-UX60A-MB-5ST, X2 ATWINC1500_MR210PA, X3 32.768

Commit message: Add directional buttons, conect pins to MCU, delete scr file
Parts:
- added C1, C10, C2, C8: 0.1uF, rcl:C0603
- added C11, C12, C13: 2.2uF, rcl:C0603
- added C14: 4.7uF, rcl:C0603
- added C15: 22uF, rcl:C0603
- added C9: (no value), rcl:C0603
- added D6: PMEG4010EGWX, CardReader:SOD123
- added L1: 4.7uH, CardReader:L0805
- added R14: 5.62k 1%, rcl:R0603
- added R15: 1.87k 1%, rcl:R0603
- added R16: 10k, rcl:R0603
- added S1: PTS645SK50SMTR92, CardReader:PTS645SK50SMTR92
- added S2, S3, S4, S5: TL1000F160Q, CardReader:TL1100
- added T1: (no value), CardReader:SOT-23
- added U5: NHD-C12832A1Z-FSW-FBW-3V3, CardReader:NHD-C12832A1Z-FSW-FBW-3V3
- added U6: MIC2288YD5-TR, CardReader:TSOT-23-5
- J1: value 5-PIN_2MM-V -> UE27AC54100; device RoboJackets-Connectors:2MM-5-V -> CardReader:USB-A
- R6, R8: value 100k -> 100k 1%
- moved J1 209.6 mm to (-41.0, -170.0)
- renumbered U$2 to J4, U$3 to U1, X1 to J3, X2 to U4
Connections:
- net N$12 renamed 3V3_EN
- removed net N$11: J1.1
- removed net N$13: J4.CD1
- removed net VCC: J2.1, R13.2, R6.1, R7.2, U3.1
- new net BOOST_ENABLE: R16.1, T1.1, U6.4
- new net BOOST_FB: R14.1, R15.2, U6.3
- new net BOOST_SW: D6.A, L1.2, U6.1
- new net BTN-DOWN: S3.1, S3.2, U1.28
- new net BTN-LEFT: S4.1, S4.2, U1.29
- new net BTN-RIGHT: S5.1, S5.2, U1.26
- new net BTN-UP: S2.1, S2.2, U1.27
- new net N$19: C1.1, U5.V0
- new net N$20: C8.1, U5.V2
- new net N$21: C10.1, U5.V3
- new net N$22: C2.1, U5.V1
- new net N$23: C9.1, U5.V4
- new net N$24: C11.1, U5.C2+
- new net N$25: C11.2, U5.C2-
- new net N$26: C13.1, U5.V_OUT
- new net N$27: C12.1
- new net N$28: C12.2, U5.C1-
- new net N$29: C3.1, J3.1
- new net SCR-!CS: U1.25, U5.!CS1
- new net SCR-!RST: U1.24, U5.!RST
- new net SCR-REG: U1.16, U5.A0
- new net SD-!CD: J4.CD1, U1.14
- new net USB-HOST-EN: U1.41
- new net VBATT: C14.1, J2.1, L1.1, R13.2, R16.2, R6.1, R7.2, U3.1, U6.5
- new net VBUS: C15.1, D6.C, J1.1, R14.2
- net !RESET: now also S1.1, S1.2
- net +3.3V: now also U5.LED+, U5.V_DD
- net +5V: now also T1.3; no longer C3.1, J3.1
- net GND: now also C1.2, C10.2, C13.2, C14.2, C15.2, C2.2, C8.2, C9.2, J1.MT1, J1.MT2, R15.1, S1.3, S1.4, S2.3, S2.4, S3.3, S3.4, S4.3, S4.4, S5.3, S5.4, T1.2, U5.LED-, U5.V_SS, U6.2; no longer J1.5
- net MOSI: now also U5.SI
- net SCK: now also U5.SCL
- net SD-!CS: now also U1.12; no longer U1.11
- net WIFI-!CS: now also U1.11; no longer U1.23
- net WIFI-!IRQ: now also U1.30
- net WIFI-CHIP-EN: now also U1.23
- net WIFI-WAKE: now also U1.15
