File: card.sch (EAGLE design)
At the start: 33 parts, among them J1 5-PIN_2MM-V, J2 B2PS-VH(LF)(SN), U3 TLV70233DBVR, X1 MINI-USB-UX60A-MB-5ST, X2 ATWINC1500_MR210PA, X3 32.768

Commit message: Add directional buttons, conect pins to MCU, delete scr file
Parts:
- removed U$3: ATSAMD21J_QFN, lib-card:ATSAMD21J_QFN
- removed X2: ATWINC1500_MR210PA, lib-card:ATWINC1500_MR210PA
- added C1, C10, C2, C8: 0.1uF, rcl:C-USC0603
- added C11, C12, C13: 2.2uF, rcl:C-USC0603
- added C14: 4.7uF, rcl:C-USC0603
- added C15: 22uF, rcl:C-USC0603
- added C9: (no value), rcl:C-USC0603
- added D6: PMEG4010EGWX, CardReader:SCHOTTKEY-DIODE-SOD123
- added L1: 4.7uH, CardReader:L-US-0805
- added R14: 5.62k 1%, rcl:R-US_R0603
- added R15: 1.87k 1%, rcl:R-US_R0603
- added R16: 10k, rcl:R-US_R0603
- added S1: PTS645SK50SMTR92, CardReader:PTS645SK50SMTR92
- added S2, S3, S4, S5: TL1000F160Q, CardReader:TL1000F160Q
- added T1: (no value), CardReader:BSS138
- added U1: ATSAMD21J_QFN, lib-card:ATSAMD21J_QFN
- added U4: ATWINC1500_MR210PA, lib-card:ATWINC1500_MR210PA
- added U5: NHD-C12832A1Z-FSW-FBW-3V3, CardReader:NHD-C12832A1Z-FSW-FBW-3V3
- added U6: MIC2288YD5-TR, CardReader:MIC2288YD5-TR
- J1: value 5-PIN_2MM-V -> UE27AC54100; device RoboJackets-Connectors:5-PIN_2MM-V -> CardReader:UE27AC54100
- R6, R8: value 100k -> 100k 1%
- renumbered U$2 to J4, X1 to J3
Connections:
- net N$12 renamed 3V3_EN
- removed net N$11: J1.1
- removed net N$13: J4.CARD_DETECT
- removed net VCC: J2.1, R13.2, R6.1, R7.2, U3.VIN
- new net BOOST_ENABLE: R16.1, T1.D, U6.EN
- new net BOOST_FB: R14.1, R15.2, U6.FB
- new net BOOST_SW: D6.A, L1.2, U6.SW
- new net BTN-DOWN: S3.1, U1.PA19/I3/SERCOM1+3.3/I2SD0
- new net BTN-LEFT: S4.1, U1.PA20/I4/SERCOM3+5.2/I2SSC
- new net BTN-RIGHT: S5.1, U1.PA17/I2C/I1/SERCOM1+3.1
- new net BTN-UP: S2.1, U1.PA18/I2/SERCOM1+3.2
- new net N$19: C1.1, U5.V0
- new net N$20: C8.1, U5.V2
- new net N$21: C10.1, U5.V3
- new net N$22: C2.1, U5.V1
- new net N$23: C9.1, U5.V4
- new net N$24: C11.1, U5.C2+
- new net N$25: C11.2, U5.C2-
- new net N$26: C13.1, U5.V_OUT
- new net N$27: C12.1
- new net N$28: C12.2, U5.C1-
- new net N$29: C3.1, J3.1
- new net SCR-!CS: U1.PA16/I2C/I0/SERCOM1+3.0, U5.!CS1
- new net SCR-!RST: U1.PA15/I15/SERCOM3+4.3, U5.!RST
- new net SCR-REG: U1.PA11/I11/AIN19/SERCOM0+2.3/I2SF0, U5.A0
- new net SD-!CD: J4.CARD_DETECT, U1.PA09/I2C/I9/AIN17/SERCOM0+2.1/I2SMC
- new net USB-HOST-EN: U1.PA28/I8
- new net VBATT: C14.1, J2.1, L1.1, R13.2, R16.2, R6.1, R7.2, U3.VIN, U6.VIN
- new net VBUS: C15.1, D6.C, J1.+5V, R14.2
- net !RESET: now also S1.1, U1.!RESET; no longer U$3.!RESET
- net +3.3V: now also U1.VDDA, U1.VDDIN, U1.VDDIO, U4.SPI_CFG, U4.VBAT, U4.VDDIO, U5.LED+, U5.V_DD; no longer U$3.VDDA, U$3.VDDIN, U$3.VDDIO, X2.SPI_CFG, X2.VBAT, X2.VDDIO
- net +5V: now also T1.G; no longer C3.1, J3.1
- net BATT-MONITOR: now also U1.PA04/EINT4/VREFB/AIN4/SERCOM0.0; no longer U$3.PA04/EINT4/VREFB/AIN4/SERCOM0.0
- net D+: now also J1.D+, U1.PA25/I13/SERCOM3+5.3/D+; no longer J1.3, U$3.PA25/I13/SERCOM3+5.3/D+
- net D-: now also J1.D-, U1.PA24/I12/SERCOM3+5.2/D-; no longer J1.2, U$3.PA24/I12/SERCOM3+5.2/D-
- net GND: now also C1.2, C10.2, C13.2, C14.2, C15.2, C2.2, C8.2, C9.2, J1.GND, J1.MT1, J1.MT2, R15.1, S1.2, S2.2, S3.2, S4.2, S5.2, T1.S, U1.GND, U1.GNDA, U4.GND, U4.GND@1, U4.GND@2, U5.LED-, U5.V_SS, U6.GND; no longer J1.4, J1.5, U$3.GND, U$3.GNDA, X2.GND, X2.GND@1, X2.GND@2
- net MISO: now also U1.PA12/I12/I2C/SERCOM2+4.0, U4.MISO; no longer U$3.PA12/I12/I2C/SERCOM2+4.0, X2.MISO
- net MOSI: now also U1.PB10/I10/SERCOM4.2/I2SMC, U4.MOSI, U5.SI; no longer U$3.PB10/I10/SERCOM4.2/I2SMC, X2.MOSI
- net N$10: now also U4.GPIO15; no longer X2.GPIO15
- net N$14: now also U1.VDDCORE; no longer U$3.VDDCORE
- net N$15: now also U1.PA00/EINT0/SERCOM1.0; no longer U$3.PA00/EINT0/SERCOM1.0
- net N$16: now also U1.PA01/EINT1/SERCOM1.1; no longer U$3.PA01/EINT1/SERCOM1.1
- net N$9: now also U4.GPIO16; no longer X2.GPIO16
- net SCK: now also U1.PB11/I11/SERCOM4.3/I2SCL, U4.SCK, U5.SCL; no longer U$3.PB11/I11/SERCOM4.3/I2SCL, X2.SCK
- net SD-!CS: now also U1.PA07/I7/AIN7/SERCOM0.3/I2SD0; no longer U$3.PA06/EINT6/AIN6/SERCOM0.2
- net WIFI-!CS: now also U1.PA06/EINT6/AIN6/SERCOM0.2, U4.CS; no longer U$3.PA14/I14/SERCOM2+4.2, X2.CS
- net WIFI-!IRQ: now also U1.PA21/I5/SERCOM3+5.3/I2SFS0, U4.!IRQ; no longer X2.!IRQ
- net WIFI-!RESET: now also U1.PA08/I2C/AIN16/SERCOM0+2.0/I2SD1, U4.!RESET; no longer U$3.PA08/I2C/AIN16/SERCOM0+2.0/I2SD1, X2.!RESET
- net WIFI-CHIP-EN: now also U1.PA14/I14/SERCOM2+4.2, U4.CHIP_EN; no longer X2.CHIP_EN
- net WIFI-WAKE: now also U1.PA10/I10/AIN18/SERCOM0+2.2/I2SCK, U4.WAKE; no longer X2.WAKE
Other:
- note added: "5V Boost Converter"
- note added: "Directional Buttons"
- note added: "LCD Display"
- note added: "Power Switch Connector"
- note added: "Wifi"
- note removed: "Add reset button"
- moved on the sheet: C5, C6, C7, D4, D5, R10, R11, R12, R9, X3
