File: hardware/card.brd (EAGLE design)
At the start: 97 x 71 mm, 93 parts, among them J1 UE27AC54100, J2 MICROSD, J3 0541323062, J4 6-PIN_2MM-V, J5 JST_2PIN, J6 B2PS-VH(LF)(SN), J7 MINI-USB-UX60A-MB-5ST, J8 JST_2PIN, U1 ATSAMD21J_QFN, U2 TS3USB221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

Commit message: fix a cap with the wrong footprint
Parts:
- C7: device rcl:C0805 -> card:C0603
Changed lines of the file:
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@@
 <attribute name="VALUE" x="75.655" y="30.385" size="1.27" layer="28" rot="MR270"/>
 </element>
-<element name="C7" library="rcl" library_urn="urn:adsk.eagle:library:334" package="C0805" package3d_urn="urn:adsk.eagle:package:23617/2" value="10uF" x="43" y="10.25" smashed="yes" rot="MR180">
+<element name="C7" library="card" package="C0603" value="10uF" x="43" y="10.25" smashed="yes" rot="MR180">
 <attribute name="NAME" x="42.48" y="12.48" size="1" layer="26" rot="MR180"/>
 <attribute name="VALUE" x="41.73" y="12.79" size="1.27" layer="28" rot="MR180"/>
@@
 <contactref element="R9" pad="1"/>
 <wire x1="41.6" y1="8.6" x2="41.6" y2="-7.75" width="0.5" layer="16"/>
-<wire x1="42.05" y1="9.05" x2="42.05" y2="10.25" width="0.5" layer="16"/>
+<wire x1="42.05" y1="9.05" x2="42.15" y2="10.25" width="0.5" layer="16"/>
 <wire x1="42.05" y1="9.05" x2="41.6" y2="8.6" width="0.5" layer="16"/>
 <contactref element="D9" pad="A"/>
@@
 <wire x1="30" y1="53.75" x2="32" y2="53.75" width="0.3" layer="1"/>
 <wire x1="30" y1="53.75" x2="28" y2="53.75" width="0.3" layer="1"/>
-<wire x1="42.05" y1="10.25" x2="42.05" y2="23.45" width="0.5" layer="16"/>
+<wire x1="42.15" y1="10.25" x2="42.05" y2="23.45" width="0.5" layer="16"/>
 <wire x1="42.05" y1="23.45" x2="41.25" y2="24.25" width="0.5" layer="16"/>
 <wire x1="41.25" y1="24.25" x2="41.25" y2="25.5" width="0.5" layer="16"/>

Commit message: exported gerbers
swapped the power switch connector
Parts:
- added J10: (no value), RoboJackets-Connectors:1X2
- added R24: 1k, rcl:R0603
- J6: value B2PS-VH(LF)(SN) -> JST_2PIN; device RoboJackets-Connectors:B2PS-CENTERED -> CardReader:JSTPH2
- moved J6 4.43 mm to (41.2, 52.5), turned to 0 degrees
- moved R21 1.27 mm to (41.3, 51.7)
- moved C5 0.25 mm to (71.8, 34.2)
- moved R1 0.25 mm to (74.0, 34.2)
- moved R2 0.25 mm to (76.2, 34.2)
- moved X2 0.25 mm to (67.8, 31.2)
Connections:
- new net SWCLK: J10.1, R24.1, U1.45
- new net SWDIO: J10.2, U1.46
- net +3.3V: now also R24.2
- net BATT: now also J6.1; no longer J6.2
- net VBATT: now also J6.2; no longer J6.1
Routing:
- net SWCLK: track 0.00 -> 15.3 mm
- net SWDIO: track 0.00 -> 14.7 mm
- net +3.3V: track 151.2 -> 157.9 mm
- net GND: track 15.8 -> 11.8 mm
- net VBATT: track 98.8 -> 102.2 mm, vias 3 -> 5
- net BATT: track 31.8 -> 34.7 mm, vias 0 -> 1
- net !RESET: track 70.5 -> 71.7 mm
Other:
- board text added: "PROGRAMMING CHARGING"
- board text added: "switch"
